File: half-moon-earring.sch (EAGLE design)
At the start: 10 parts, among them IC1 TTP223

Commit message: bom list
Parts:
- PW1: value CR2025 -> CR2025 BATERY HOLDER
- R1, R2: value 150 -> 150R
- T1: value (none) -> BC817
- renumbered U$1 to PW1, U$2 to LED2, U$3 to LED3, U$4 to LED1
Changed lines of the file:
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@@
 <part name="GND4" library="supply1" library_urn="urn:adsk.eagle:library:371" deviceset="GND" device=""/>
 <part name="P+2" library="supply1" library_urn="urn:adsk.eagle:library:371" deviceset="VCC" device=""/>
-<part name="T1" library="transistor" library_urn="urn:adsk.eagle:library:402" deviceset="*-NPN-" device="SOT23-BEC" package3d_urn="urn:adsk.eagle:package:28748/2" technology="BC817-16LT1"/>
+<part name="T1" library="transistor" library_urn="urn:adsk.eagle:library:402" deviceset="*-NPN-" device="SOT23-BEC" package3d_urn="urn:adsk.eagle:package:28748/2" technology="BC817-16LT1" value="BC817"/>
 <part name="GND1" library="supply1" library_urn="urn:adsk.eagle:library:371" deviceset="GND" device=""/>
-<part name="R1" library="rcl" library_urn="urn:adsk.eagle:library:334" deviceset="R-EU_" device="M0805" package3d_urn="urn:adsk.eagle:package:23556/2" value="150"/>
-<part name="R2" library="rcl" library_urn="urn:adsk.eagle:library:334" deviceset="R-EU_" device="M0805" package3d_urn="urn:adsk.eagle:package:23556/2" value="150"/>
-<part name="U$1" library="supply1" deviceset="CR2025" device=""/>
+<part name="R1" library="rcl" library_urn="urn:adsk.eagle:library:334" deviceset="R-EU_" device="M0805" package3d_urn="urn:adsk.eagle:package:23556/2" value="150R"/>
+<part name="R2" library="rcl" library_urn="urn:adsk.eagle:library:334" deviceset="R-EU_" device="M0805" package3d_urn="urn:adsk.eagle:package:23556/2" value="150R"/>
+<part name="PW1" library="supply1" deviceset="CR2025" device="" value="CR2025 BATERY HOLDER"/>
 <part name="P+3" library="supply1" library_urn="urn:adsk.eagle:library:371" deviceset="VCC" device=""/>
 <part name="GND5" library="supply1" library_urn="urn:adsk.eagle:library:371" deviceset="GND" device=""/>
-<part name="U$2" library="Eletroblocks Lib" deviceset="LED5050" device=""/>
-<part name="U$3" library="Eletroblocks Lib" deviceset="LED5050" device=""/>
-<part name="U$4" library="Eletroblocks Lib" deviceset="LED5050" device=""/>
+<part name="LED2" library="Eletroblocks Lib" deviceset="LED5050" device=""/>
+<part name="LED3" library="Eletroblocks Lib" deviceset="LED5050" device=""/>
+<part name="LED1" library="Eletroblocks Lib" deviceset="LED5050" device=""/>
 <part name="P+4" library="supply1" library_urn="urn:adsk.eagle:library:371" deviceset="VCC" device=""/>
 </parts>
@@
 <instance part="T1" gate="G$1" x="40.64" y="-48.26" smashed="yes" grouprefs="DRIVER1">
 <attribute name="NAME" x="43.18" y="-48.26" size="1.778" layer="95"/>
-<attribute name="VALUE" x="30.48" y="-43.18" size="1.778" layer="96"/>
+<attribute name="VALUE" x="48.26" y="-50.8" size="1.778" layer="96" rot="R90"/>
 </instance>
 <instance part="GND1" gate="1" x="43.18" y="-58.42" smashed="yes" grouprefs="DRIVER1">
@@
 <attribute name="VALUE" x="46.482" y="-39.37" size="1.778" layer="96" rot="R90"/>
 </instance>
-<instance part="U$1" gate="G$1" x="10.16" y="73.66" smashed="yes" grouprefs="SOURCE"/>
+<instance part="PW1" gate="G$1" x="10.16" y="73.66" smashed="yes" grouprefs="SOURCE"/>
 <instance part="P+3" gate="VCC" x="10.16" y="96.52" smashed="yes" grouprefs="SOURCE">
 <attribute name="VALUE" x="7.62" y="93.98" size="1.778" layer="96" rot="R90"/>
@@
 <attribute name="VALUE" x="7.62" y="48.26" size="1.778" layer="96"/>
 </instance>
-<instance part="U$2" gate="G$1" x="20.32" y="-99.06" smashed="yes" grouprefs="LEDS">
+<instance part="LED2" gate="G$1" x="20.32" y="-99.06" smashed="yes" grouprefs="LEDS">
 <attribute name="NAME" x="25.4" y="-101.6" size="1.778" layer="95"/>
 <attribute name="VALUE" x="25.4" y="-104.14" size="1.778" layer="96"/>
 </instance>
-<instance part="U$3" gate="G$1" x="20.32" y="-109.22" smashed="yes" grouprefs="LEDS">
+<instance part="LED3" gate="G$1" x="20.32" y="-109.22" smashed="yes" grouprefs="LEDS">
 <attribute name="NAME" x="25.4" y="-111.76" size="1.778" layer="95"/>
 <attribute name="VALUE" x="25.4" y="-114.3" size="1.778" layer="96"/>
 </instance>
-<instance part="U$4" gate="G$1" x="20.32" y="-88.9" smashed="yes" grouprefs="LEDS">
+<instance part="LED1" gate="G$1" x="20.32" y="-88.9" smashed="yes" grouprefs="LEDS">
 <attribute name="NAME" x="25.4" y="-91.44" size="1.778" layer="95"/>
 <attribute name="VALUE" x="25.4" y="-93.98" size="1.778" layer="96"/>
@@
 </segment>
 <segment>
-<pinref part="U$1" gate="G$1" pin="P$2"/>
+<pinref part="PW1" gate="G$1" pin="P$2"/>
 <pinref part="GND5" gate="1" pin="GND"/>
 <wire x1="10.16" y1="66.04" x2="10.16" y2="53.34" width="0.1524" layer="91" grouprefs="SOURCE"/>
@@
 </segment>
 <segment>
-<pinref part="U$1" gate="G$1" pin="P$1"/>
+<pinref part="PW1" gate="G$1" pin="P$1"/>
 <pinref part="P+3" gate="VCC" pin="VCC"/>
 <wire x1="10.16" y1="78.74" x2="10.16" y2="93.98" width="0.1524" layer="91" grouprefs="SOURCE"/>
 </segment>
 <segment>
-<pinref part="U$3" gate="G$1" pin="P$1"/>
+<pinref part="LED3" gate="G$1" pin="P$1"/>
 <wire x1="20.32" y1="-109.22" x2="12.7" y2="-109.22" width="0.1524" layer="91" grouprefs="LEDS"/>
 <wire x1="12.7" y1="-109.22" x2="12.7" y2="-99.06" width="0.1524" layer="91" grouprefs="LEDS"/>
-<pinref part="U$2" gate="G$1" pin="P$1"/>
+<pinref part="LED2" gate="G$1" pin="P$1"/>
 <wire x1="20.32" y1="-99.06" x2="12.7" y2="-99.06" width="0.1524" layer="91" grouprefs="LEDS"/>
 <wire x1="12.7" y1="-99.06" x2="12.7" y2="-88.9" width="0.1524" layer="91" grouprefs="LEDS"/>
-<pinref part="U$4" gate="G$1" pin="P$1"/>
+<pinref part="LED1" gate="G$1" pin="P$1"/>
 <wire x1="12.7" y1="-88.9" x2="20.32" y2="-88.9" width="0.1524" layer="91" grouprefs="LEDS"/>
 <pinref part="P+4" gate="VCC" pin="VCC"/>
@@
 </segment>
 <segment>
-<pinref part="U$4" gate="G$1" pin="P$2"/>
+<pinref part="LED1" gate="G$1" pin="P$2"/>
 <wire x1="25.4" y1="-88.9" x2="38.1" y2="-88.9" width="0.1524" layer="91" grouprefs="LEDS"/>
 <wire x1="38.1" y1="-88.9" x2="38.1" y2="-99.06" width="0.1524" layer="91" grouprefs="LEDS"/>
-<pinref part="U$3" gate="G$1" pin="P$2"/>
+<pinref part="LED3" gate="G$1" pin="P$2"/>
 <wire x1="38.1" y1="-99.06" x2="38.1" y2="-109.22" width="0.1524" layer="91" grouprefs="LEDS"/>
 <wire x1="38.1" y1="-109.22" x2="25.4" y2="-109.22" width="0.1524" layer="91" grouprefs="LEDS"/>
-<pinref part="U$2" gate="G$1" pin="P$2"/>
+<pinref part="LED2" gate="G$1" pin="P$2"/>
 <wire x1="25.4" y1="-99.06" x2="38.1" y2="-99.06" width="0.1524" layer="91" grouprefs="LEDS"/>
 <junction x="38.1" y="-99.06" grouprefs="LEDS"/>

Commit message: correção de tamanho
Parts:
- removed PW1: CR2025 BATERY HOLDER, supply1:CR2025
- added U$1: CR2035, cr2025:CR2035
Connections:
- net GND: now also U$1.P$2; no longer PW1.P$2
- net VCC: now also U$1.P$1; no longer PW1.P$1
Changed lines of the file:
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@@
 <?xml version="1.0" encoding="utf-8"?>
 <!DOCTYPE eagle SYSTEM "eagle.dtd">
-<eagle version="9.5.2">
+<eagle version="9.6.2">
 <drawing>
 <settings>
@@
 <part name="R1" library="rcl" library_urn="urn:adsk.eagle:library:334" deviceset="R-EU_" device="M0805" package3d_urn="urn:adsk.eagle:package:23556/2" value="150R"/>
 <part name="R2" library="rcl" library_urn="urn:adsk.eagle:library:334" deviceset="R-EU_" device="M0805" package3d_urn="urn:adsk.eagle:package:23556/2" value="150R"/>
-<part name="PW1" library="supply1" deviceset="CR2025" device="" value="CR2025 BATERY HOLDER"/>
-<part name="P+3" library="supply1" library_urn="urn:adsk.eagle:library:371" deviceset="VCC" device=""/>
-<part name="GND5" library="supply1" library_urn="urn:adsk.eagle:library:371" deviceset="GND" device=""/>
 <part name="LED2" library="Eletroblocks Lib" deviceset="LED5050" device=""/>
 <part name="LED3" library="Eletroblocks Lib" deviceset="LED5050" device=""/>
 <part name="LED1" library="Eletroblocks Lib" deviceset="LED5050" device=""/>
 <part name="P+4" library="supply1" library_urn="urn:adsk.eagle:library:371" deviceset="VCC" device=""/>
+<part name="U$1" library="cr2025" deviceset="CR2035" device=""/>
+<part name="P+5" library="supply1" library_urn="urn:adsk.eagle:library:371" deviceset="VCC" device=""/>
+<part name="GND6" library="supply1" library_urn="urn:adsk.eagle:library:371" deviceset="GND" device=""/>
 </parts>
 <sheets>
@@
 <attribute name="VALUE" x="46.482" y="-39.37" size="1.778" layer="96" rot="R90"/>
 </instance>
-<instance part="PW1" gate="G$1" x="10.16" y="73.66" smashed="yes" grouprefs="SOURCE"/>
-<instance part="P+3" gate="VCC" x="10.16" y="96.52" smashed="yes" grouprefs="SOURCE">
-<attribute name="VALUE" x="7.62" y="93.98" size="1.778" layer="96" rot="R90"/>
-</instance>
-<instance part="GND5" gate="1" x="10.16" y="50.8" smashed="yes" grouprefs="SOURCE">
-<attribute name="VALUE" x="7.62" y="48.26" size="1.778" layer="96"/>
-</instance>
 <instance part="LED2" gate="G$1" x="20.32" y="-99.06" smashed="yes" grouprefs="LEDS">
 <attribute name="NAME" x="25.4" y="-101.6" size="1.778" layer="95"/>
@@
 <instance part="P+4" gate="VCC" x="12.7" y="-81.28" smashed="yes" grouprefs="LEDS">
 <attribute name="VALUE" x="10.16" y="-83.82" size="1.778" layer="96" rot="R90"/>
+</instance>
+<instance part="U$1" gate="G$1" x="10.16" y="66.04" smashed="yes" grouprefs="SOURCE"/>
+<instance part="P+5" gate="VCC" x="10.16" y="78.74" smashed="yes" grouprefs="SOURCE">
+<attribute name="VALUE" x="7.62" y="76.2" size="1.778" layer="96" rot="R90"/>
+</instance>
+<instance part="GND6" gate="1" x="10.16" y="50.8" smashed="yes" grouprefs="SOURCE">
+<attribute name="VALUE" x="7.62" y="48.26" size="1.778" layer="96"/>
 </instance>
 </instances>
@@
 </segment>
 <segment>
-<pinref part="PW1" gate="G$1" pin="P$2"/>
-<pinref part="GND5" gate="1" pin="GND"/>
-<wire x1="10.16" y1="66.04" x2="10.16" y2="53.34" width="0.1524" layer="91" grouprefs="SOURCE"/>
+<pinref part="U$1" gate="G$1" pin="P$2"/>
+<pinref part="GND6" gate="1" pin="GND"/>
+<wire x1="10.16" y1="58.42" x2="10.16" y2="53.34" width="0.1524" layer="91" grouprefs="SOURCE"/>
 </segment>
 </net>
@@
 <wire x1="35.56" y1="25.4" x2="35.56" y2="22.86" width="0.1524" layer="91" grouprefs="TOUCH1"/>
 <wire x1="35.56" y1="22.86" x2="58.42" y2="22.86" width="0.1524" layer="91" grouprefs="TOUCH1"/>
-</segment>
-<segment>
-<pinref part="PW1" gate="G$1" pin="P$1"/>
-<pinref part="P+3" gate="VCC" pin="VCC"/>
-<wire x1="10.16" y1="78.74" x2="10.16" y2="93.98" width="0.1524" layer="91" grouprefs="SOURCE"/>
 </segment>
 <segment>
@@
 <junction x="12.7" y="-99.06" grouprefs="LEDS"/>
 </segment>
+<segment>
+<pinref part="P+5" gate="VCC" pin="VCC"/>
+<pinref part="U$1" gate="G$1" pin="P$1"/>
+<wire x1="10.16" y1="76.2" x2="10.16" y2="71.12" width="0.1524" layer="91" grouprefs="SOURCE"/>
+</segment>
 </net>
